Commit message: Fix the error

File: project4/workspace/catkin_ws/src/my_robot/urdf/my_robot.xacro (robot description, xacro)
@@ -118,5 +118,5 @@
     <dynamics damping="1.0" friction="1.0"/>
   </joint>
-  <link name='camera'>
+  <link name='camera_link'>
     <inertial>
       <mass value="0.1"/>
@@ -128,5 +128,5 @@
       />
     </inertial>
-    <collision name='camera_collision'>
+    <collision name='camera_link_collision'>
       <origin xyz="0 0 0" rpy=" 0 0 0"/>
       <geometry>
@@ -134,5 +134,5 @@
       </geometry>
     </collision>
-    <visual name='camera_visual'>
+    <visual name='camera_link_visual'>
       <origin xyz="0 0 0" rpy=" 0 0 0"/>
       <geometry>
@@ -141,7 +141,7 @@
     </visual>
   </link>
-  <joint type="fixed" name="camera_hinge">
+  <joint type="fixed" name="camera_joint">
     <origin xyz="0.2 0 0" rpy="0 0 0"/>
-    <child link="camera"/>
+    <child link="camera_link"/>
     <parent link="chassis"/>
     <axis xyz="0 1 0" rpy="0 0 0"/>
